File: AstroPix_telescope.kicad_sch (KiCad schematic)
At the start: 13 parts, among them J1 AstroPix2_pcie, J2 AstroPix2_pcie, J3 AstroPix2_pcie, J4 AstroPix2_pcie, P1 pcie_GECCO

Commit message: Added Logo + minor improvements
Parts:
- added Logo1: KIT_logo, astropix:logo, symbol astropix:KIT_logo
- P1: footprint Connector_PCBEdge:BUS_PCIexpress_x16 -> astropix:BUS_PCIexpress_x16_mod
Other:
- note added: "Weak pulldown on MISO right, allows telescope to be operated with less than 4 layers"
- moved on the sheet: J2, J3, J4, R1, R2, R3, R4, R5, R6

Commit message: Added signal thPMOS, viastitching and removed unused rings
Connections:
- net DAC_blpix: no longer J1.B32 (DAC_blpix), J2.B32 (DAC_blpix), J3.B32 (DAC_blpix), J4.B32 (DAC_blpix)
- net DAC_ThPMOS: now reaches P1.A32 (C4_1)
- net DAC_ThPMOS: now also J1.B32 (DAC_blpix), J2.B32 (DAC_blpix), J3.B32 (DAC_blpix), J4.B32 (DAC_blpix)
- no-connect marks 57 -> 56
Other:
- note added: "Added THPMOS for v3"

Commit message: Added VSSA for Astropix3
Parts:
- P1: footprint astropix:BUS_PCIexpress_x16_mod -> astropix:pcie_astropix
Connections:
- net VSSA: now reaches P1.B10 (POW8)
- net VSSA: now also J1.A10 (POW8), J1.A9 (POW8), J1.B10 (POW8), J1.B9 (POW8), J2.A10 (POW8), J2.A9 (POW8), J2.B10 (POW8), J2.B9 (POW8), J3.A10 (POW8), J3.A9 (POW8), J3.B10 (POW8), J3.B9 (POW8), J4.A10 (POW8), J4.A9 (POW8), J4.B10 (POW8), J4.B9 (POW8), P1.B9 (POW8)
- no-connect marks 56 -> 54
