File: AstroPix_telescope.kicad_sch (KiCad schematic)
At the start: 14 parts, among them J1 AstroPix2_pcie, J2 AstroPix2_pcie, J3 AstroPix2_pcie, J4 AstroPix2_pcie, P1 pcie_GECCO

Commit message: Preliminary design...
Parts:
- added JP1: VDDJP, Connector_PinHeader_2.54mm:PinHeader_1x03_P2.54mm_Vertical, symbol Jumper:Jumper_3_Bridged12
- added Logo2: ~, astropix:SCIPP_Logo, symbol astropix:SCIPP_Logo
- added Logo3: ANL_LOGO, astropix:ANL_Logo, symbol AstropixTriggerLib:ANL_LOGO
- P1: footprint astropix:pcie_astropix -> astropix:BUS_PCIexpress_x16_mod
- R1, R2, R3, R4, R5, R6: now not fitted
Connections:
- net sr_out is gone; now on net sr_out1: J1.A22 (sr_out), J2.B25 (sr_sin)
- net -HV: no longer P1.A1 (HV), P1.B1 (HV)
- net DAC_ThPix: no longer J1.A34 (DAC_ThPix), J2.A34 (DAC_ThPix), J3.A34 (DAC_ThPix), J4.A34 (DAC_ThPix)
- net DAC_VCasc2!: no longer J1.A33 (DAC_Vcasc2), J2.A33 (DAC_Vcasc2), J3.A33 (DAC_Vcasc2), J4.A33 (DAC_Vcasc2)
- net DAC_vminuspix: no longer J1.A35 (DAC_vminuspix), J2.A35 (DAC_vminuspix), J3.A35 (DAC_vminuspix), J4.A35 (DAC_vminuspix)
- net POW4_in: now also JP1.1 (A)
- net VDD18_in: now also JP1.3 (B)
- net VSSA: now also P1.A5 (VSSA), P1.A6 (VSSA); no longer P1.B10 (POW8), P1.B9 (POW8)
- net spi1_clk: no longer J1.B40 (spi_right_clk)
- net spi1_csn: no longer J1.B43 (spi_right_csn)
- net spi1_miso0: no longer J1.B42 (spi_right_miso0)
- net spi1_miso1: no longer J1.B41 (spi_right_miso1)
- net spi1_mosi: no longer J1.B44 (spi_right_mosi)
- net spi2_clk: no longer J2.B40 (spi_right_clk)
- net spi2_csn: no longer J2.B43 (spi_right_csn)
- net spi2_miso0: no longer J2.B42 (spi_right_miso0)
- net spi2_miso1: no longer J2.B41 (spi_right_miso1)
- net spi2_mosi: no longer J2.B44 (spi_right_mosi)
- net spi3_clk: no longer J3.B40 (spi_right_clk)
- net spi3_csn: no longer J3.B43 (spi_right_csn)
- net spi3_miso0: no longer J3.B42 (spi_right_miso0)
- net spi3_miso1: no longer J3.B41 (spi_right_miso1)
- net spi3_mosi: no longer J3.B44 (spi_right_mosi)
- net spi_right_clk: no longer J4.B40 (spi_right_clk)
- net spi_right_csn: no longer J4.B43 (spi_right_csn)
- net spi_right_miso0: no longer J4.B42 (spi_right_miso0)
- net spi_right_miso1: no longer J4.B41 (spi_right_miso1)
- net spi_right_mosi: no longer J4.B44 (spi_right_mosi)
- net sr_out1: no longer J2.A22 (sr_out), J3.B25 (sr_sin)
- net sr_out2: now also J2.A22 (sr_out), J3.B25 (sr_sin); no longer J3.A22 (sr_out), J4.B25 (sr_sin)
- net sr_out3: now also J3.A22 (sr_out), J4.B25 (sr_sin); no longer J4.A22 (sr_out), P1.A22 (FMC_LA17_CC_P)
- net sample_clk0_N renamed DigInj
- net DigInj: now also J1.B40 (DIgInj), J2.B40 (DIgInj), J3.B40 (DIgInj), J4.B40 (DIgInj); no longer J1.B19 (sample_clk_N)
- net sample_clk0_P: no longer names the net of P1.B41 (FMC_LA16_N)
- net sample_clk0_P: no longer J1.B18 (sample_clk_P)
- net sample_clk1_N renamed sample_clk_N
- net sample_clk_N: now also J1.B19 (sample_clk_N), J2.B19 (sample_clk_N), J3.B19 (sample_clk_N), J4.B19 (sample_clk_N)
- net sample_clk1_P renamed sample_clk_P
- net sample_clk_P: now also J1.B18 (sample_clk_P), J2.B18 (sample_clk_P), J3.B18 (sample_clk_P), J4.B18 (sample_clk_P)
- net sample_clk2_N: no longer names the net of P1.B42 (FMC_LA14_P)
- net sample_clk2_N: no longer J2.B19 (sample_clk_N)
- net sample_clk2_P: no longer names the net of P1.B43 (FMC_LA14_N)
- net sample_clk2_P: no longer J2.B18 (sample_clk_P)
- net sample_clk3_N: no longer names the net of P1.B44 (FMC_LA12_P)
- net sample_clk3_N: no longer J3.B19 (sample_clk_N)
- net sample_clk3_P: no longer names the net of P1.B45 (FMC_LA12_N)
- net sample_clk3_P: no longer J3.B18 (sample_clk_P)
- net sample_clk4_N: no longer names the net of P1.B46 (FMC_LA10_P)
- net sample_clk4_N: no longer J4.B19 (sample_clk_N)
- net sample_clk4_P: no longer names the net of P1.B47 (FMC_LA10_N)
- net sample_clk4_P: no longer J4.B18 (sample_clk_P)
- new net VDD: JP1.2 (C)
- new net sr_out4: J4.A22 (sr_out), P1.A22 (FMC_LA17_CC_P)
- no-connect marks 54 -> 63
Other:
- moved on the sheet: H1, H2, P1

Commit message: V3 initial commit for fabrication.
Other:
- note added: "Mounting Holes & Logos"
- note added: "PCI-e GECCO Goldfinger"
- note added: "PCI-e slots for Astropix Carrier Boards"
- note added: "Pull down resistors: Not used in A-STEP (Astropix V3)"
- company: Nicolas Striebig, KIT ADL -> KIT ADL, ANL, UCSC
- title: AstroPix Telescope -> AstroPix Telescope V3
- moved on the sheet: H1, H2, JP1, P1
