File: AstroPix_telescope.kicad_pcb (KiCad board)
At the start: 4 copper layers, 84.3 x 120.9 mm, 46 parts, among them J1 AstroPix2_pcie, J1 Conn_01x06, J2 AstroPix2_pcie, J2 EPK.00.250.NTN, J3 AstroPix2_pcie, J4 AstroPix2_pcie, P1 pcie_GECCO, U1 74AVCH2T45,125, U2 TLV70013DDCR

Commit message: New revision.
Parts:
- removed C1 (x2), C4 (x2), C5 (x2): 10uF, Capacitor_SMD:C_0603_1608Metric_Pad1.08x0.95mm_HandSolder
- removed C2 (x2), C3 (x2): 1uF, Capacitor_SMD:C_0603_1608Metric_Pad1.08x0.95mm_HandSolder
- removed G1 (x2): ANL_LOGO, Astropix Trigger:ANL_Logo
- removed the J1 at (158.1, 44.8)
- removed the J1 at (133.3, 32.2)
- removed the J2 at (183.6, 38.2)
- removed the J2 at (107.8, 38.8)
- removed L1 (x2): 10nH, Inductor_SMD:L_0603_1608Metric_Pad1.05x0.95mm_HandSolder
- removed the R1 at (178.6, 40.0)
- removed the R1 at (112.8, 37.0)
- removed the R2 at (162.4, 38.6)
- removed the R2 at (129.0, 38.4)
- removed TPAtlas1 (x2): TP_Atlas_TRIG, Astropix Trigger:TP420X150
- removed TPFPGA1 (x2): TP_FPGA_TRIG, Astropix Trigger:TP420X150
- removed TPGND1 (x2): TP_GND, Astropix Trigger:TP420X150
- removed U1 (x2): 74AVCH2T45,125, Package_SO:VSSOP-8_2.3x2mm_P0.5mm
- removed U2 (x2): TLV70013DDCR, Package_TO_SOT_SMD:TSOT-23-5_HandSoldering
- added REF**: ANL_Logo, astropix:ANL_Logo, F.Cu at (122.4, 141.3)
- added REF**: SCIPP_Logo, astropix:SCIPP_Logo, F.Cu at (129.0, 143.8)
Routing:
- net (no net): track 62.6 -> 0.00 mm
- net GND: vias 142 -> 10
- removed copper zone on F.Cu, net (none)
Other:
- board size 84.3 x 120.9 mm -> 84.4 x 97.1 mm
- board text added: "AstroPix Telescope 1.1.1"
- board text added: "UCSC SCIPP"
- board text removed: "Argonne National Laboratory"
- board text removed: "AstroPix Telescope 1.1"
- board text removed: "Astropix Trigger V1.0"
- board text removed: "DNP"
- board text removed: "UCSC-SCIPP"
- board text removed: "University of California: Santa Cruz"

Commit message: Preliminary design...
Parts:
- removed REF**: ANL_Logo, astropix:ANL_Logo
- removed REF**: SCIPP_Logo, astropix:SCIPP_Logo
- added JP1: VDDJP, Connector_PinHeader_2.54mm:PinHeader_1x03_P2.54mm_Vertical, F.Cu at (106.4, 137.2)
- added Logo2: ~, astropix:SCIPP_Logo, F.Cu at (183.0, 145.8)
- added Logo3: ANL_LOGO, astropix:ANL_Logo, F.Cu at (176.7, 147.2)
- P1: footprint Connector_PCBEdge:BUS_PCIexpress_x16 -> astropix:BUS_PCIexpress_x16_mod
- moved Logo1 54.9 mm to (164.2, 142.5)
Connections:
- J1 pad A22: /sr_out -> /sr_out1
- J1 pad A33: /DAC_VCasc2! -> (no net)
- J1 pad A34: /DAC_ThPix -> (no net)
- J1 pad A35: /DAC_vminuspix -> (no net)
- J1 pad B18: /sample_clk0_P -> /sample_clk_P
- J1 pad B19: /sample_clk0_N -> /sample_clk_N
- J1 pad B40: /spi1_clk -> /DigInj
- J1 pad B41: /spi1_miso1 -> (no net)
- J1 pad B42: /spi1_miso0 -> (no net)
- J1 pad B43: /spi1_csn -> (no net)
- J1 pad B44: /spi1_mosi -> (no net)
- J2 pad A22: /sr_out1 -> /sr_out2
- J2 pad A33: /DAC_VCasc2! -> (no net)
- J2 pad A34: /DAC_ThPix -> (no net)
- J2 pad A35: /DAC_vminuspix -> (no net)
- J2 pad B18: /sample_clk2_P -> /sample_clk_P
- J2 pad B19: /sample_clk2_N -> /sample_clk_N
- J2 pad B25: /sr_out -> /sr_out1
- J2 pad B40: /spi2_clk -> /DigInj
- J2 pad B41: /spi2_miso1 -> (no net)
- J2 pad B42: /spi2_miso0 -> (no net)
- J2 pad B43: /spi2_csn -> (no net)
- J2 pad B44: /spi2_mosi -> (no net)
- J3 pad A22: /sr_out2 -> /sr_out3
- J3 pad A33: /DAC_VCasc2! -> (no net)
- J3 pad A34: /DAC_ThPix -> (no net)
- J3 pad A35: /DAC_vminuspix -> (no net)
- J3 pad B18: /sample_clk3_P -> /sample_clk_P
- J3 pad B19: /sample_clk3_N -> /sample_clk_N
- J3 pad B25: /sr_out1 -> /sr_out2
- J3 pad B40: /spi3_clk -> /DigInj
- J3 pad B41: /spi3_miso1 -> (no net)
- J3 pad B42: /spi3_miso0 -> (no net)
- J3 pad B43: /spi3_csn -> (no net)
- J3 pad B44: /spi3_mosi -> (no net)
- J4 pad A22: /sr_out3 -> /sr_out4
- J4 pad A33: /DAC_VCasc2! -> (no net)
- J4 pad A34: /DAC_ThPix -> (no net)
- J4 pad A35: /DAC_vminuspix -> (no net)
- J4 pad B18: /sample_clk4_P -> /sample_clk_P
- J4 pad B19: /sample_clk4_N -> /sample_clk_N
- J4 pad B25: /sr_out2 -> /sr_out3
- J4 pad B40: /spi_right_clk -> /DigInj
- J4 pad B41: /spi_right_miso1 -> (no net)
- J4 pad B42: /spi_right_miso0 -> (no net)
- J4 pad B43: /spi_right_csn -> (no net)
- J4 pad B44: /spi_right_mosi -> (no net)
- P1 pad A1: -HV -> unconnected-(P1-HV-PadA1)
- P1 pad A22: /sr_out3 -> /sr_out4
- P1 pad A5: unconnected-(P1-PadA5) -> VSSA
- P1 pad A6: unconnected-(P1-PadA6) -> VSSA
- P1 pad B1: -HV -> unconnected-(P1-HV-PadB1)
- P1 pad B10: VSSA -> unconnected-(P1-POW8-PadB10)
- P1 pad B18: /sample_clk1_P -> /sample_clk_P
- P1 pad B19: /sample_clk1_N -> /sample_clk_N
- P1 pad B40: /sample_clk0_N -> /DigInj
- P1 pad B41: /sample_clk0_P -> unconnected-(P1-FMC_LA16_N-PadB41)
- P1 pad B42: /sample_clk2_N -> unconnected-(P1-FMC_LA14_P-PadB42)
- P1 pad B43: /sample_clk2_P -> unconnected-(P1-FMC_LA14_N-PadB43)
- P1 pad B44: /sample_clk3_N -> unconnected-(P1-FMC_LA12_P-PadB44)
- P1 pad B45: /sample_clk3_P -> unconnected-(P1-FMC_LA12_N-PadB45)
- P1 pad B46: /sample_clk4_N -> unconnected-(P1-FMC_LA10_P-PadB46)
- P1 pad B47: /sample_clk4_P -> unconnected-(P1-FMC_LA10_N-PadB47)
- P1 pad B9: VSSA -> unconnected-(P1-POW8-PadB9)
Routing:
- net /sample_clk0_P: track 165.5 -> 0.00 mm
- net /sample_clk0_N: track 165.5 -> 0.00 mm
- net /sample_clk4_P: track 165.4 -> 0.00 mm
- net /sample_clk4_N: track 165.4 -> 0.00 mm
- net /sample_clk2_P: track 165.3 -> 0.00 mm
- net /sample_clk2_N: track 165.2 -> 0.00 mm
- net /sample_clk3_N: track 164.6 -> 0.00 mm
- net /sample_clk3_P: track 164.5 -> 0.00 mm
- net /sr_out4: track 0.00 -> 122.7 mm, vias 0 -> 2
- net /sample_clk_P: track 0.00 -> 110.2 mm, vias 0 -> 2
- net /sample_clk_N: track 0.00 -> 108.9 mm, vias 0 -> 2
- net /DigInj: track 0.00 -> 101.2 mm
- net /sr_out3: track 122.8 -> 27.8 mm, vias 2 -> 0
- net -HV: track 98.1 -> 62.5 mm, vias 1 -> 0
- net /sr_out: track 27.9 -> 0.00 mm
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- removed copper zone on B.Cu, net /POW4_in
- removed copper zone on B.Cu, net /VDD18_in
- removed copper zone on F.Cu, net VSSA
Other:
- board text added: "1:POW4 3:VDD18"
- board text added: "AstroPix Telescope 1.3 for Astropix v3"
- board text added: "VDDJP"
- board text removed: "AstroPix Telescope 1.1.1"

Commit message: V3 initial commit for fabrication.
Routing:
- net /spi3_miso0: track 45.4 -> 39.7 mm, vias 2 -> 1
- net /spi1_miso1: track 43.3 -> 38.5 mm
- net /spi3_miso1: track 39.8 -> 37.0 mm, vias 2 -> 1
- net /spi2_csn: track 38.8 -> 36.2 mm
- net /spi2_clk: track 40.9 -> 38.3 mm
- net GND: track 6.82 -> 9.18 mm, vias 149 -> 200
- net /spi3_clk: track 45.4 -> 43.6 mm
- net /spi2_mosi: track 38.2 -> 36.5 mm, vias 1 -> 0
- net /Inj: track 93.4 -> 95.0 mm
- net /spi3_mosi: track 39.1 -> 40.6 mm, vias 1 -> 0
- net /spi1_csn: track 38.0 -> 36.6 mm
- net /spi1_mosi: track 39.9 -> 41.2 mm
- net /spi_left_miso1: track 31.2 -> 32.4 mm
- net /spi_left_clk: track 33.0 -> 34.1 mm
- net /spi_left_csn: track 31.0 -> 31.9 mm
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